Commit message: update

File: install/aircraft_design/share/aircraft_design/urdf/aircraft.urdf.xacro (robot description, xacro)
@@ -1,61 +1 @@
-<?xml version="1.0"?>
-<robot xmlns:xacro="http://www.ros.org/wiki/xacro" name="aircraft">
-    <xacro:property name="L_2" value="8.781" />
-    <xacro:property name="L_landing" value="4.10" />
-    <xacro:property name="PI" value="3.14159265359" />
-    <link name="aircraft_nose_wheel_link">
-        <visual>
-            <origin xyz="0 0 0" rpy="0 0 0"/>
-            <geometry>
-                <mesh filename="package://aircraft_design/meshes/aircraft_nose_wheel.stl" scale="1 1 1"/>
-            </geometry>
-            <material name="black">
-                <color rgba="0.1 0.1 0.1 1.0"/>
-            </material>
-        </visual>
-    </link>
-    <link name="aircraft_base_link">
-        <visual>
-            <origin xyz="0 0 0" rpy="0 -0.06 ${PI}"/>
-            <geometry>
-                <mesh filename="package://aircraft_design/meshes/aircraft_base.stl" scale="1 1 1"/>
-            </geometry>
-            <material name="white">
-                <color rgba="0.9 0.9 0.9 1.0"/>
-            </material>
-        </visual>
-    </link>
-    <link name="aircraft_left_mlg_link">
-        <visual>
-            <origin xyz="0 0 0" rpy="0 0 0"/>
-            <geometry>
-                <mesh filename="package://aircraft_design/meshes/aircraft_left_mlg.stl" scale="1 1 1"/>
-            </geometry>
-            <material name="black"/>
-        </visual>
-    </link>
-    <link name="aircraft_right_mlg_link">
-        <visual>
-            <origin xyz="0 0 0" rpy="0 0 0"/>
-            <geometry>
-                <mesh filename="package://aircraft_design/meshes/aircraft_right_mlg.stl" scale="1 1 1"/>
-            </geometry>
-            <material name="black"/>
-        </visual>
-    </link>
-    <joint name="aircraft_nose_to_base" type="fixed">
-        <parent link="aircraft_nose_wheel_link"/>
-        <child link="aircraft_base_link"/>
-        <origin xyz="-${L_2} 0 0" rpy="0 0 0"/>
-    </joint>
-    <joint name="aircraft_base_to_left_mlg" type="fixed">
-        <parent link="aircraft_base_link"/>
-        <child link="aircraft_left_mlg_link"/>
-        <origin xyz="0 -${L_landing/2} 0" rpy="0 0 0"/>
-    </joint>
-    <joint name="aircraft_base_to_right_mlg" type="fixed">
-        <parent link="aircraft_base_link"/>
-        <child link="aircraft_right_mlg_link"/>
-        <origin xyz="0 ${L_landing/2} 0" rpy="0 0 0"/>
-    </joint>
-</robot>
+/home/student/flight_ws/build/aircraft_design/urdf/aircraft.urdf.xacro

File: install/aircraft_design/share/aircraft_design/urdf/system.urdf.xacro (robot description, xacro)
@@ -1,11 +1 @@
-<?xml version="1.0"?>
-<robot xmlns:xacro="http://www.ros.org/wiki/xacro" name="pushback_system">
-    <xacro:include filename="$(find aircraft_design)/urdf/tractor.urdf.xacro" />
-    <xacro:include filename="$(find aircraft_design)/urdf/aircraft.urdf.xacro" />
-    <joint name="tow_joint" type="continuous">
-        <parent link="tractor_hitch_link"/>
-        <child link="aircraft_nose_wheel_link"/>
-        <origin xyz="0 0 0" rpy="0 0 0"/>
-        <axis xyz="0 0 1"/>
-    </joint>
-</robot>
+/home/student/flight_ws/build/aircraft_design/urdf/system.urdf.xacro

File: install/aircraft_design/share/aircraft_design/urdf/tractor.urdf.xacro (robot description, xacro)
@@ -1,24 +1 @@
-<?xml version="1.0"?>
-<robot xmlns:xacro="http://www.ros.org/wiki/xacro" name="tractor">
-    <link name="tractor_base_link">
-        <visual>
-            <geometry><mesh filename="package://aircraft_design/meshes/tractor_base.stl" scale="1 1 1"/></geometry>
-            <material name="dark_grey"><color rgba="0.2 0.2 0.2 1.0"/></material>
-        </visual>
-        <visual>
-            <geometry><mesh filename="package://aircraft_design/meshes/rear_wheel_group.stl" scale="1 1 1"/></geometry>
-            <material name="black"><color rgba="0.1 0.1 0.1 1.0"/></material>
-        </visual>
-    </link>
-    <link name="tractor_hitch_link">
-        <visual>
-            <geometry><mesh filename="package://aircraft_design/meshes/tractor_hitch.stl" scale="1 1 1"/></geometry>
-            <material name="grey"><color rgba="0.6 0.6 0.6 1.0"/></material>
-        </visual>
-    </link>
-    <joint name="tractor_base_to_hitch" type="fixed">
-        <parent link="tractor_base_link"/>
-        <child link="tractor_hitch_link"/>
-        <origin xyz="0 0 0.255" rpy="0 0 0"/>
-    </joint>
-</robot>
+/home/student/flight_ws/build/aircraft_design/urdf/tractor.urdf.xacro

File: src/aircraft_design/urdf/aircraft.urdf.xacro (robot description, xacro)
@@ -1,10 +1,11 @@
 <?xml version="1.0"?>
 <robot xmlns:xacro="http://www.ros.org/wiki/xacro" name="aircraft">
-    <xacro:property name="L_2" value="8.781" />
+    <xacro:property name="L_2" value="8.4" />
     <xacro:property name="L_landing" value="4.10" />
     <xacro:property name="PI" value="3.14159265359" />
+    <xacro:property name="dz" value="0.200302" />
     <link name="aircraft_nose_wheel_link">
         <visual>
-            <origin xyz="0 0 0" rpy="0 0 0"/>
+            <origin xyz="0 0 ${dz}" rpy="0 0 0"/>
             <geometry>
                 <mesh filename="package://aircraft_design/meshes/aircraft_nose_wheel.stl" scale="1 1 1"/>
@@ -17,5 +18,5 @@
     <link name="aircraft_base_link">
         <visual>
-            <origin xyz="0 0 0" rpy="0 -0.06 ${PI}"/>
+            <origin xyz="0 0 0" rpy="0 0.02 0"/>
             <geometry>
                 <mesh filename="package://aircraft_design/meshes/aircraft_base.stl" scale="1 1 1"/>
@@ -47,15 +48,15 @@
         <parent link="aircraft_nose_wheel_link"/>
         <child link="aircraft_base_link"/>
-        <origin xyz="-${L_2} 0 0" rpy="0 0 0"/>
+        <origin xyz="-${L_2} 0 ${dz}" rpy="0 0 0"/>
     </joint>
     <joint name="aircraft_base_to_left_mlg" type="fixed">
         <parent link="aircraft_base_link"/>
         <child link="aircraft_left_mlg_link"/>
-        <origin xyz="0 -${L_landing/2} 0" rpy="0 0 0"/>
+        <origin xyz="0 ${L_landing/2} 0" rpy="0 0 0"/>
     </joint>
     <joint name="aircraft_base_to_right_mlg" type="fixed">
         <parent link="aircraft_base_link"/>
         <child link="aircraft_right_mlg_link"/>
-        <origin xyz="0 ${L_landing/2} 0" rpy="0 0 0"/>
+        <origin xyz="0 -${L_landing/2} 0" rpy="0 0 0"/>
     </joint>
 </robot>

File: src/aircraft_design/urdf/tractor.urdf.xacro (robot description, xacro)
@@ -20,5 +20,5 @@
         <parent link="tractor_base_link"/>
         <child link="tractor_hitch_link"/>
-        <origin xyz="0 0 0.255" rpy="0 0 0"/>
+        <origin xyz="0 0 0" rpy="0 0 0"/>
     </joint>
 </robot>
