Commit message: testing

File: src/aircraft_design/urdf/system.urdf.xacro (robot description, xacro)
@@ -6,5 +6,5 @@
         <parent link="tractor_hitch_link"/>
         <child link="aircraft_nose_wheel_link"/>
-        <origin xyz="0 0 0.20028" rpy="0 0 0"/>
+        <origin xyz="0 0 0.31626" rpy="0 0 0"/>
         <axis xyz="0 0 1"/>
     </joint>
