Commit message: update

File: src/aircraft_design/urdf/aircraft.urdf.xacro (robot description, xacro)
@@ -1,11 +1,26 @@
 <?xml version="1.0"?>
 <robot xmlns:xacro="http://www.ros.org/wiki/xacro" name="aircraft">
-    <xacro:property name="L_2" value="8.4" />
-    <xacro:property name="L_landing" value="4.10" />
+    <!-- ===================================================================== -->
+    <!-- 1. PHYSICAL & KINEMATIC PARAMETERS                                    -->
+    <!-- Derived directly from the Blender CAD measurements.                   -->
+    <!-- ===================================================================== -->
+    <!-- L_2: Longitudinal distance from Nose Axle to Main Landing Gear (MLG) Axle -->
+    <xacro:property name="L_2" value="8.146" />
+    <!-- L_landing: Total track width (Y-axis offset between Left & Right MLG) -->
+    <!-- 2.01545m left + 2.01545m right = 4.0309m -->
+    <xacro:property name="L_landing" value="4.0309" />
     <xacro:property name="PI" value="3.14159265359" />
-    <xacro:property name="dz" value="0.200302" />
+    <!-- dz: Vertical height difference between the Nose Axle and MLG Axle -->
+    <!-- MLG axle is higher (+Z relative to nose wheel axle) -->
+    <xacro:property name="dz" value="0.1515" />
+    <!-- ===================================================================== -->
+    <!-- 2. LINK DEFINITIONS                                                   -->
+    <!-- All visual origins stay at (0,0,0) with (0,0,0) rotation    -->
+    <!-- because the origins and pitch were permanently made into the STLs!   -->
+    <!-- ===================================================================== -->
+    <!-- NOSE WHEEL LINK (Parent link for the aircraft chain) -->
     <link name="aircraft_nose_wheel_link">
         <visual>
-            <origin xyz="0 0 ${dz}" rpy="0 0 0"/>
+            <origin xyz="0 0 0" rpy="0 0 0"/>
             <geometry>
                 <mesh filename="package://aircraft_design/meshes/aircraft_nose_wheel.stl" scale="1 1 1"/>
@@ -16,7 +31,8 @@
         </visual>
     </link>
+    <!-- MAIN FUSELAGE / BASE LINK -->
     <link name="aircraft_base_link">
         <visual>
-            <origin xyz="0 0 0" rpy="0 0.02 0"/>
+            <origin xyz="0 0 0" rpy="0 0 0"/>
             <geometry>
                 <mesh filename="package://aircraft_design/meshes/aircraft_base.stl" scale="1 1 1"/>
@@ -27,4 +43,5 @@
         </visual>
     </link>
+    <!-- LEFT MAIN LANDING GEAR -->
     <link name="aircraft_left_mlg_link">
         <visual>
@@ -36,4 +53,5 @@
         </visual>
     </link>
+    <!-- RIGHT MAIN LANDING GEAR -->
     <link name="aircraft_right_mlg_link">
         <visual>
@@ -45,18 +63,28 @@
         </visual>
     </link>
+    <!-- ===================================================================== -->
+    <!-- 3. JOINT DEFINITIONS                                                  -->
+    <!-- Tree structure: tractor_hitch -> nose_wheel -> base_link -> MLGs      -->
+    <!-- ===================================================================== -->
+    <!-- JOINT: Nose Wheel to Base Link -->
+    <!-- Base link is BEHIND (-X) and HIGHER (+Z) than the nose wheel axle. -->
     <joint name="aircraft_nose_to_base" type="fixed">
         <parent link="aircraft_nose_wheel_link"/>
         <child link="aircraft_base_link"/>
-        <origin xyz="-${L_2} 0 ${dz}" rpy="0 0 0"/>
+        <origin xyz="-${L_2} -0.031327 ${dz}" rpy="0 0 0"/>
     </joint>
+    <!-- JOINT: Base Link to Left Main Landing Gear -->
     <joint name="aircraft_base_to_left_mlg" type="fixed">
         <parent link="aircraft_base_link"/>
         <child link="aircraft_left_mlg_link"/>
         <origin xyz="0 ${L_landing/2} 0" rpy="0 0 0"/>
+        <axis xyz="0 1 0"/>
     </joint>
+    <!-- JOINT: Base Link to Right Main Landing Gear -->
     <joint name="aircraft_base_to_right_mlg" type="fixed">
         <parent link="aircraft_base_link"/>
         <child link="aircraft_right_mlg_link"/>
         <origin xyz="0 -${L_landing/2} 0" rpy="0 0 0"/>
+        <axis xyz="0 1 0"/>
     </joint>
 </robot>

File: src/aircraft_design/urdf/system.urdf.xacro (robot description, xacro)
@@ -6,5 +6,5 @@
         <parent link="tractor_hitch_link"/>
         <child link="aircraft_nose_wheel_link"/>
-        <origin xyz="0 0 0" rpy="0 0 0"/>
+        <origin xyz="0 0 0.20028" rpy="0 0 0"/>
         <axis xyz="0 0 1"/>
     </joint>

File: src/aircraft_design/urdf/tractor.urdf.xacro (robot description, xacro)
@@ -1,24 +1,61 @@
 <?xml version="1.0"?>
 <robot xmlns:xacro="http://www.ros.org/wiki/xacro" name="tractor">
+    <!-- ===================================================================== -->
+    <!-- 1. MATERIAL DEFINITIONS                                               -->
+    <!-- Declared globally so they can be reused cleanly across the file.      -->
+    <!-- ===================================================================== -->
+    <material name="dark_grey">
+        <color rgba="0.2 0.2 0.2 1.0"/>
+    </material>
+    <material name="black">
+        <color rgba="0.1 0.1 0.1 1.0"/>
+    </material>
+    <material name="grey">
+        <color rgba="0.6 0.6 0.6 1.0"/>
+    </material>
+    <!-- ===================================================================== -->
+    <!-- 2. LINK DEFINITIONS                                                   -->
+    <!-- ===================================================================== -->
+    <!-- TRACTOR BASE LINK (Main Body & Rear Wheels) -->
+    <!-- This serves as the root link for the tractor's kinematic chain. -->
     <link name="tractor_base_link">
+        <!-- Tractor Chassis Visual -->
         <visual>
-            <geometry><mesh filename="package://aircraft_design/meshes/tractor_base.stl" scale="1 1 1"/></geometry>
-            <material name="dark_grey"><color rgba="0.2 0.2 0.2 1.0"/></material>
+            <origin xyz="0 0 0" rpy="0 0 0"/>
+            <geometry>
+                <mesh filename="package://aircraft_design/meshes/tractor_base.stl" scale="1 1 1"/>
+            </geometry>
+            <material name="dark_grey"/>
         </visual>
+        <!-- Rear Wheels Visual -->
+        <!-- Grouped into the base_link visually to minimize TF overhead -->
         <visual>
-            <geometry><mesh filename="package://aircraft_design/meshes/rear_wheel_group.stl" scale="1 1 1"/></geometry>
-            <material name="black"><color rgba="0.1 0.1 0.1 1.0"/></material>
+            <origin xyz="0 0 0" rpy="0 0 0"/>
+            <geometry>
+                <mesh filename="package://aircraft_design/meshes/rear_wheel_group.stl" scale="1 1 1"/>
+            </geometry>
+            <material name="black"/>
         </visual>
     </link>
+    <!-- TRACTOR HITCH LINK (Clamping Mechanism) -->
+    <!-- This acts as the dynamic attachment point for the aircraft_nose_wheel_link -->
     <link name="tractor_hitch_link">
         <visual>
-            <geometry><mesh filename="package://aircraft_design/meshes/tractor_hitch.stl" scale="1 1 1"/></geometry>
-            <material name="grey"><color rgba="0.6 0.6 0.6 1.0"/></material>
+            <origin xyz="0 0 0" rpy="0 0 0"/>
+            <geometry>
+                <mesh filename="package://aircraft_design/meshes/tractor_hitch.stl" scale="1 1 1"/>
+            </geometry>
+            <material name="grey"/>
         </visual>
     </link>
+    <!-- ===================================================================== -->
+    <!-- 3. JOINT DEFINITIONS                                                  -->
+    <!-- ===================================================================== -->
+    <!-- JOINT: Tractor Base to Hitch -->
+    <!-- Places the hitch clamping mechanism exactly 0.023m forward on the X-axis -->
     <joint name="tractor_base_to_hitch" type="fixed">
         <parent link="tractor_base_link"/>
         <child link="tractor_hitch_link"/>
-        <origin xyz="0 0 0" rpy="0 0 0"/>
+        <origin xyz="0.023 0 0" rpy="0 0 0"/>
     </joint>
 </robot>

Commit message: update

File: src/aircraft_design/urdf/aircraft.urdf.xacro (robot description, xacro)
@@ -1,19 +1,5 @@
 <?xml version="1.0"?>
 <robot xmlns:xacro="http://www.ros.org/wiki/xacro" name="aircraft">
-    <!-- ===================================================================== -->
-    <!-- 1. PHYSICAL & KINEMATIC PARAMETERS                                    -->
-    <!-- Derived directly from the Blender CAD measurements.                   -->
-    <!-- ===================================================================== -->
-    <!-- L_2: Longitudinal distance from Nose Axle to Main Landing Gear (MLG) Axle -->
-    <xacro:property name="L_2" value="8.146" />
-    <!-- L_landing: Total track width (Y-axis offset between Left & Right MLG) -->
-    <!-- 2.01545m left + 2.01545m right = 4.0309m -->
-    <xacro:property name="L_landing" value="4.0309" />
-    <xacro:property name="PI" value="3.14159265359" />
-    <!-- dz: Vertical height difference between the Nose Axle and MLG Axle -->
-    <!-- MLG axle is higher (+Z relative to nose wheel axle) -->
-    <xacro:property name="dz" value="0.1515" />
-    <!-- ===================================================================== -->
-    <!-- 2. LINK DEFINITIONS                                                   -->
+    <!-- 1. LINK DEFINITIONS                                                   -->
     <!-- All visual origins stay at (0,0,0) with (0,0,0) rotation    -->
     <!-- because the origins and pitch were permanently made into the STLs!   -->
@@ -64,13 +50,12 @@
     </link>
     <!-- ===================================================================== -->
-    <!-- 3. JOINT DEFINITIONS                                                  -->
+    <!-- 2. JOINT DEFINITIONS                                                  -->
     <!-- Tree structure: tractor_hitch -> nose_wheel -> base_link -> MLGs      -->
     <!-- ===================================================================== -->
     <!-- JOINT: Nose Wheel to Base Link -->
-    <!-- Base link is BEHIND (-X) and HIGHER (+Z) than the nose wheel axle. -->
     <joint name="aircraft_nose_to_base" type="fixed">
         <parent link="aircraft_nose_wheel_link"/>
         <child link="aircraft_base_link"/>
-        <origin xyz="-${L_2} -0.031327 ${dz}" rpy="0 0 0"/>
+        <origin xyz="0 0 0" rpy="0 0 0"/>
     </joint>
     <!-- JOINT: Base Link to Left Main Landing Gear -->
@@ -78,5 +63,5 @@
         <parent link="aircraft_base_link"/>
         <child link="aircraft_left_mlg_link"/>
-        <origin xyz="0 ${L_landing/2} 0" rpy="0 0 0"/>
+        <origin xyz="0 0 0" rpy="0 0 0"/>
         <axis xyz="0 1 0"/>
     </joint>
@@ -85,5 +70,5 @@
         <parent link="aircraft_base_link"/>
         <child link="aircraft_right_mlg_link"/>
-        <origin xyz="0 -${L_landing/2} 0" rpy="0 0 0"/>
+        <origin xyz="0 0 0" rpy="0 0 0"/>
         <axis xyz="0 1 0"/>
     </joint>

File: src/aircraft_design/urdf/system.urdf.xacro (robot description, xacro)
@@ -6,5 +6,5 @@
         <parent link="tractor_hitch_link"/>
         <child link="aircraft_nose_wheel_link"/>
-        <origin xyz="0 0 0.31626" rpy="0 0 0"/>
+        <origin xyz="-8.146 0 0" rpy="0 0 0"/>
         <axis xyz="0 0 1"/>
     </joint>
